Commit message: Update simple_gripper.urdf

File: my_gripper/simple_gripper.urdf (robot description, URDF)
Before this commit: robot simple_gripper, 2 links, 1 joints
Links:
- removed link right_leg
- added link left_finger, mass 0.1; collision box size=0.025 0.075 0.025; visual box size=0.025 0.075 0.025
- added link left_finger_tip, mass 0.1; collision box size=0.025 0.05 0.025; visual box size=0.025 0.05 0.025
- added link palm, mass 0.5; collision box size=0.025 0.05 0.025; visual box size=0.025 0.05 0.025
- added link right_finger, mass 0.1; collision box size=0.025 0.075 0.025; visual box size=0.025 0.075 0.025
- added link right_finger_tip, mass 0.1; collision box size=0.025 0.05 0.025; visual box size=0.025 0.05 0.025
- link riser: mass None -> 10; geometry collision box size=0.025 0.025 0.25; visual box size=0.025 0.025 0.25
Joints:
- removed joint base_to_right_leg
- added joint left_finger_tip: type revolute, parent left_finger, child left_finger_tip, origin xyz=0 0.025 0 rpy=0 0 0, axis 0 0 1, limit lower=-0.4 upper=0.4
- added joint palm_left_finger: type revolute, parent palm, child left_finger, origin xyz=0 -0.025 0 rpy=0 0 0, axis 0 0 1, limit lower=-0.4 upper=0.4
- added joint palm_right_finger: type revolute, parent palm, child right_finger, origin xyz=0 0.025 0 rpy=0 0 0, axis 0 0 1, limit lower=-0.4 upper=0.4
- added joint palm_riser: type prismatic, parent riser, child palm, axis 0 0 1, limit lower=0 upper=0.9
- added joint right_finger_tip: type revolute, parent right_finger, child right_finger_tip, origin xyz=0 0.025 0 rpy=0 0 0, axis 0 0 1, limit lower=-0.4 upper=0.4
