Commit message: Update my_gripper.xacro

File: my_gripper/my_gripper.xacro (robot description, xacro)
@@ -2,5 +2,5 @@
 <robot xmlns:xacro="http://ros.org/wiki/xacro">
   <!-- Main gripper link -->
-  <xacro:macro name="my_gripper_macro"
+  <xacro:macro name="my_gripper_macro">
   <material name="blue">
       <color rgba="0 0 0.8 1"/>

Commit message: Update my_gripper.xacro

File: my_gripper/my_gripper.xacro (robot description, xacro)
@@ -12,4 +12,9 @@
       <color rgba="1 1 1 1"/>
     </material>
+    <joint name="base1_joint" type="fixed">
+      <origin xyz="0 0 -0.1302" rpy="0 0 0" />
+      <parent link="base_link"/>
+      <child link="riser" />
+    </joint>
     <link name="riser">
       <visual>
@@ -41,5 +46,5 @@
           <box size="0.025 0.05 0.025"/>
         </geometry>
-        <origin rpy="0 0 0" xyz="0 0 0.0125"/>
+        <origin rpy="0 0 0" xyz="0 0 2.0125"/>
       </collision>
       <inertial>
@@ -126,5 +131,5 @@
     <joint name="palm_left_finger" type="revolute">
       <axis xyz="0 0 1"/>
-      <limit lower="-0.4" upper="0.4"/>
+      <limit lower="-0.4" upper="0.4" effort="2.5" velocity="1.0"/>
       <origin rpy="0 0 0" xyz="0 -0.025 0"/>
       <parent link="palm"/>
@@ -133,5 +138,5 @@
     <joint name="left_finger_tip" type="revolute">
       <axis xyz="0 0 1"/>
-      <limit lower="-0.4" upper="0.4"/>
+      <limit lower="-0.4" upper="0.4" effort="2.5" velocity="1.0"/>
       <origin rpy="0 0 0" xyz="0 0.025 0"/>
       <parent link="left_finger"/>
@@ -140,5 +145,5 @@
     <joint name="palm_right_finger" type="revolute">
       <axis xyz="0 0 1"/>
-      <limit lower="-0.4" upper="0.4"/>
+      <limit lower="-0.4" upper="0.4" effort="2.5" velocity="1.0"/>
       <origin rpy="0 0 0" xyz="0 0.025 0"/>
       <parent link="palm"/>
@@ -147,5 +152,5 @@
     <joint name="right_finger_tip" type="revolute">
       <axis xyz="0 0 1"/>
-      <limit lower="-0.4" upper="0.4"/>
+      <limit lower="-0.4" upper="0.4" effort="2.5" velocity="1.0"/>
       <origin rpy="0 0 0" xyz="0 0.025 0"/>
       <parent link="right_finger"/>
@@ -154,5 +159,5 @@
     <joint name="palm_riser" type="prismatic">
       <axis xyz="0 0 1"/>
-      <limit lower="0" upper="0.9"/>
+      <limit lower="0" upper="0.9" effort="2.5" velocity="1.0"/>
       <parent link="riser"/>
       <child link="palm"/>
@@ -214,3 +219,3 @@
     </plugin>
   </gazebo>
-  </robot>
+</robot>

Commit message: Update my_gripper.xacro

File: my_gripper/my_gripper.xacro (robot description, xacro)
@@ -30,5 +30,5 @@
       </collision>
       <inertial>
-        <mass value="10"/>
+        <mass value="0.2"/>
         <inertia ixx="0.01" ixy="0.0" ixz="0.0" iyy="0.01" iyz="0.0" izz="0.01"/>
       </inertial>
@@ -49,5 +49,5 @@
       </collision>
       <inertial>
-        <mass value="0.5"/>
+        <mass value="0.1"/>
         <inertia ixx="0.01" ixy="0.0" ixz="0.0" iyy="0.01" iyz="0.0" izz="0.01"/>
       </inertial>
