Commit message: Update balsa_arm.urdf

File: balsa_arm/balsa_arm_description/urdf/balsa_arm.urdf (robot description, URDF)
Before this commit: robot balsa_arm, 4 links, 3 joints
Links:
- link base_link: geometry collision box size=0.065 0.055 0.003; visual box size=0.065 0.055 0.003
Joints:
- joint elbow: axis 0 0 1 -> 0 1 0
- joint wrist: axis 0 0 1 -> 0 1 0; origin xyz=0 0 0.153 -> xyz=0 0 0.068
